File: PCB/Alarm_Clock_PCB.kicad_sch (KiCad schematic)
At the start: 11 parts, among them J1 Conn_01x08_Pin, SW1 SW_Push, SW2 SW_Push, SW3 SW_Push, SW4 SW_Push, U1 XIAO-ESP32-C3-SMD

Commit message: Changed PCB from SMD to DIP soldering
Parts:
- U1: footprint Seeed_Studio_XIAO_Series:XIAO-ESP32-C3-SMD -> Seeed_Studio_XIAO_Series:XIAO-ESP32-C3-DIP
Changed lines of the file:
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@@
 			)
 		)
-		(property "Footprint" "Seeed_Studio_XIAO_Series:XIAO-ESP32-C3-SMD"
+		(property "Footprint" "Seeed_Studio_XIAO_Series:XIAO-ESP32-C3-DIP"
 			(at 104.902 124.714 0)
 			(hide yes)
